Commit message: update sim01

File: src/sim01_urdf/urdf/urdf/corn_harvester.urdf (robot description, URDF)
Before this commit: robot cornn, 6 links, 5 joints
Links:
- link base_link: mass 40025 -> 40068; geometry collision mesh filename=package://sim01_urdf/meshes/base_link.STL; visual mesh filename=package://sim01_urdf/meshes/base_link.STL
- link laser_link: geometry collision mesh filename=package://sim01_urdf/meshes/laser_link.STL; visual mesh filename=package://sim01_urdf/meshes/laser_link.STL
- link left_front_wheel_link0: geometry collision mesh filename=package://sim01_urdf/meshes/left_front_wheel_link0.STL; visual mesh filename=package://sim01_urdf/meshes/left_front_wheel_link0.STL
- link left_rear_wheel_link3: geometry collision mesh filename=package://sim01_urdf/meshes/left_rear_wheel_link3.STL; visual mesh filename=package://sim01_urdf/meshes/left_rear_wheel_link3.STL
- link right_front_wheel_link1: geometry collision mesh filename=package://sim01_urdf/meshes/right_front_wheel_link1.STL; visual mesh filename=package://sim01_urdf/meshes/right_front_wheel_link1.STL
- link right_rear_wheel_link2: geometry collision mesh filename=package://sim01_urdf/meshes/right_rear_wheel_link2.STL; visual mesh filename=package://sim01_urdf/meshes/right_rear_wheel_link2.STL
Joints:
- joint laser_joint: origin xyz=-1.7526 -1.5139 4.9382 rpy=1.5718 -0.0036179 0.74761 -> xyz=2.8823 -3.7226 0.005493 rpy=0.0043263 0.7476 -3.1367
- joint left_front_wheel_joint0: axis 0 0 0 -> 0 1 0; origin xyz=-2.3657 -4.2754 0.033114 rpy=-1.5708 0 1.5708 -> xyz=3.4954 1.1624 2.767 rpy=0 1.5708 0
- joint left_rear_wheel_joint3: axis 0 0 0 -> 0 1 0; origin xyz=3.4943 -4.2754 0.033114 rpy=-1.5708 0 1.5708 -> xyz=-2.3646 1.1624 2.767 rpy=0 1.5708 0
- joint right_front_wheel_joint1: axis 0 0 0 -> 0 1 0; origin xyz=-2.3657 1.2587 -0.24756 rpy=-1.5708 0 -1.5708 -> xyz=3.4954 1.4431 -2.767 rpy=0 -1.5708 0
- joint right_rear_wheel_joint2: axis 0 0 0 -> 0 1 0; origin xyz=3.4943 1.2587 -0.24756 rpy=-1.5708 0 -1.5708 -> xyz=-2.3646 1.4431 -2.767 rpy=0 -1.5708 0

Commit message: update sim01

File: src/sim01_urdf/urdf/urdf/corn_harvester.urdf (robot description, URDF)
Before this commit: robot corn_harvester, 6 links, 5 joints
Joints:
- joint laser_joint: origin xyz=2.8823 -3.7226 0.005493 rpy=0.0043263 0.7476 -3.1367 -> xyz=0.005493 -2.8923 3.7226 rpy=1.5718 -0.0036179 2.3184
- joint left_front_wheel_joint0: axis 0 1 0 -> 1 0 0; origin xyz=3.4954 1.1624 2.767 rpy=0 1.5708 0 -> xyz=2.767 -3.5054 -1.1624 rpy=-1.5708 0 3.1416
- joint left_rear_wheel_joint3: axis 0 1 0 -> 1 0 0; origin xyz=-2.3646 1.1624 2.767 rpy=0 1.5708 0 -> xyz=2.767 2.3546 -1.1624 rpy=-1.5708 0 3.1416
- joint right_front_wheel_joint1: axis 0 1 0 -> 1 0 0; origin xyz=3.4954 1.4431 -2.767 rpy=0 -1.5708 0 -> xyz=-2.767 -3.5054 -1.4431 rpy=1.5708 0 0
- joint right_rear_wheel_joint2: axis 0 1 0 -> 1 0 0; origin xyz=-2.3646 1.4431 -2.767 rpy=0 -1.5708 0 -> xyz=-2.767 2.3546 -1.4431 rpy=1.5708 0 0
