Commit message: update

File: src/sim01_urdf/urdf/urdf/corn_harvester copy.urdf (robot description, URDF)
Before this commit: robot corn_harvester, 7 links, 6 joints
Links:
- link base_link: mass 10.2316767990512 -> 40068
- link laser_link: mass 0.1 -> 141.89
- link left_front_wheel_link0: mass 0.503853041294886 -> 950.62
- link left_rear_wheel_link3: mass 0.503852022031433 -> 950.62
- link right_front_wheel_link1: mass 0.503852021760132 -> 950.62
- link right_rear_wheel_link2: mass 0.503853041294886 -> 950.62
