Commit message: fix laser

File: ROS2/src/sim01_urdf/urdf/urdf/corn_harvester.urdf (robot description, URDF)
Before this commit: robot corn_harvester, 7 links, 6 joints
Links:
- link laser_link: geometry visual mesh filename=package://sim01_urdf/meshes/laser_link.STL
Joints:
- joint laser_joint: origin xyz=0.005493 -2.8923 3.7226 rpy=1.5718 -0.0036179 2.3184 -> xyz=0.005493 -2.8923 3.7226 rpy=0 -0.0036179 2.3184

File: ROS2/src/sim01_urdf/urdf/xacro/gazebo/move_control.urdf.xacro (robot description, xacro)
@@ -3,6 +3,6 @@
     <gazebo>
         <plugin
-            filename="gz-sim-diff-drive-system"
-            name="gz::sim::systems::DiffDrive">
+            filename="libignition-gazebo-diff-drive-system"
+            name="ignition::gazebo::systems::DiffDrive">
             <left_joint>left_front_wheel_joint0</left_joint>
             <left_joint>left_rear_wheel_joint3</left_joint>
@@ -27,6 +27,6 @@
     <!-- 关节状态发布 -->
     <gazebo>
-        <plugin filename="gz-sim-joint-state-publisher-system"
-        name="gz::sim::systems::JointStatePublisher">
+        <plugin filename="ignition-gazebo-joint-state-publisher-system"
+        name="ignition::gazebo::systems::JointStatePublisher">
         </plugin>
     </gazebo>

File: ROS2/src/sim01_urdf/urdf/xacro/gazebo/sensors_plugin.urdf.xacro (robot description, xacro)
@@ -3,6 +3,6 @@
     <gazebo>
         <plugin
-        filename="gz-sim-sensors-system"
-        name="gz::sim::systems::Sensors">
+        filename="libignition-gazebo-sensors-system"
+        name="ignition::gazebo::systems::Sensors">
         <render_engine>ogre2</render_engine>
         </plugin>
@@ -11,4 +11,5 @@
     <gazebo reference="laser_link">
         <sensor name='gpu_lidar' type='gpu_lidar'>
+        <pose>0 0 1.0 0 0 0</pose>   <!-- 只给激光传感器加本地偏移：x y z R P Y -->
         <topic>scan</topic>
         <update_rate>30</update_rate> <!-- 激光雷达更新频率 -->
@@ -34,7 +35,7 @@
             </range>
         </lidar>
-        <always_on>true</always_on>
+        <alwaysOn>1</alwaysOn>
         <visualize>true</visualize> <!-- 激光雷达射线是否可视化 -->
-        <pose relative_to="laser_link"/>
+        <ignition_frame_id>laser_link</ignition_frame_id>
         </sensor>
     </gazebo>

File: ROS2/src/sim03_gazebo_classic/urdf/urdf/corn_harvester.urdf (robot description, URDF)
Before this commit: robot corn_harvester, 7 links, 6 joints
Links:
- link laser_link: geometry visual mesh filename=package://sim03_gazebo_classic/meshes/laser_link.STL
Joints:
- joint laser_joint: origin xyz=0.005493 -2.8923 3.7226 rpy=1.5718 -0.0036179 2.3184 -> xyz=0.005493 -2.8923 3.7226 rpy=0 -0.0036179 2.3184

File: ROS2/src/sim03_gazebo_classic/urdf/xacro/gazebo/sensors_plugin.urdf.xacro (robot description, xacro)
@@ -5,5 +5,5 @@
       <visualize>true</visualize>
       <update_rate>10</update_rate>
-      <pose>0 0 0.075 0 0 0</pose>
+      <pose>0 0 0 0 0 0</pose>
       <ray>
           <scan>
@@ -17,5 +17,5 @@
           <range>
             <min>0.120000</min>
-            <max>3.5</max>
+            <max>20</max>
             <resolution>0.015000</resolution>
           </range>

Commit message: update new lite model

File: ROS2/src/sim01_urdf/urdf/urdf/corn_harvester.urdf (robot description, URDF)
Before this commit: robot corn_harvester, 7 links, 6 joints
Links:
- removed link base_footprint
- link base_link: mass 10.2316767990512 -> 83.037
- link laser_link: mass 0.1 -> 0; geometry collision mesh filename=package://sim01_urdf/meshes/laser_link.STL; visual mesh filename=package://sim01_urdf/meshes/laser_link.STL
- link left_front_wheel_link0: mass 0.503853041294886 -> 0.98793
- link left_rear_wheel_link3: mass 0.503852022031433 -> 0.98793
- link right_front_wheel_link1: mass 0.503852021760132 -> 0.98793
- link right_rear_wheel_link2: mass 0.503853041294886 -> 0.98793
Joints:
- removed joint base_joint
- removed joint laser_joint
- added joint laser_mount: type fixed, parent base_link, child laser_link, origin xyz=0 0.25 0.43 rpy=-1.5708 0 -1.5708, axis 0 0 0
- joint left_front_wheel_joint0: origin xyz=2.767 -3.5054 -1.1624 rpy=-1.5708 0 3.1416 -> xyz=-0.09 0.3 0.03 rpy=1.5708 0 0
- joint left_rear_wheel_joint3: origin xyz=2.767 2.3546 -1.1624 rpy=-1.5708 0 3.1416 -> xyz=-0.09 -0.3 0.03 rpy=1.5708 0 0
- joint right_front_wheel_joint1: axis 1 0 0 -> -1 0 0; origin xyz=-2.767 -3.5054 -1.4431 rpy=1.5708 0 0 -> xyz=0.09 0.3 0.03 rpy=1.5708 0 3.1416
- joint right_rear_wheel_joint2: axis 1 0 0 -> -1 0 0; origin xyz=-2.767 2.3546 -1.4431 rpy=1.5708 0 0 -> xyz=0.09 -0.3 0.03 rpy=1.5708 0 3.1416

File: ROS2/src/sim01_urdf/urdf/xacro/gazebo/move_control.urdf.xacro (robot description, xacro)
@@ -13,5 +13,5 @@
             <odom_publish_frequency>50</odom_publish_frequency>
             <frame_id>odom</frame_id>
-            <child_frame_id>base_footprint</child_frame_id>
+            <child_frame_id>base_link</child_frame_id>
             <topic>/cmd_vel</topic>
             <max_linear_acceleration>10</max_linear_acceleration>

Commit message: fix laser and wheel

File: ROS2/src/sim01_urdf/urdf/urdf/corn_harvester.urdf (robot description, URDF)
Before this commit: robot corn_harvester, 6 links, 5 joints
Links:
- added link base_footprint; visual sphere radius=0.001
- link laser_link: mass 0 -> 0.15944
Joints:
- added joint base_mount: type fixed, parent base_footprint, child base_link, origin xyz=0.0 0.0 0.06
- joint laser_mount: origin xyz=0 0.25 0.43 rpy=-1.5708 0 -1.5708 -> xyz=0 0.25 0.43 rpy=0 0 0
- joint right_front_wheel_joint1: axis -1 0 0 -> 1 0 0; origin xyz=0.09 0.3 0.03 rpy=1.5708 0 3.1416 -> xyz=0.09 0.3 0.03 rpy=-1.1331 0 3.1416
- joint right_rear_wheel_joint2: axis -1 0 0 -> 1 0 0; origin xyz=0.09 -0.3 0.03 rpy=1.5708 0 3.1416 -> xyz=0.09 -0.3 0.03 rpy=-1.1331 0 3.1416

File: ROS2/src/sim01_urdf/urdf/xacro/gazebo/move_control.urdf.xacro (robot description, xacro)
@@ -9,9 +9,9 @@
             <right_joint>right_front_wheel_joint1</right_joint>
             <right_joint>right_rear_wheel_joint2</right_joint>
-            <wheel_separation>0.4</wheel_separation>
-            <wheel_radius>0.0375</wheel_radius>
+            <wheel_separation>0.58</wheel_separation>
+            <wheel_radius>0.085</wheel_radius>
             <odom_publish_frequency>50</odom_publish_frequency>
             <frame_id>odom</frame_id>
-            <child_frame_id>base_link</child_frame_id>
+            <child_frame_id>base_footprint</child_frame_id>
             <topic>/cmd_vel</topic>
             <max_linear_acceleration>10</max_linear_acceleration>

File: ROS2/src/sim01_urdf/urdf/xacro/gazebo/sensors_plugin.urdf.xacro (robot description, xacro)
@@ -3,5 +3,5 @@
     <gazebo>
         <plugin
-        filename="libignition-gazebo-sensors-system"
+        filename="ignition-gazebo-sensors-system"
         name="ignition::gazebo::systems::Sensors">
         <render_engine>ogre2</render_engine>
@@ -11,5 +11,5 @@
     <gazebo reference="laser_link">
         <sensor name='gpu_lidar' type='gpu_lidar'>
-        <pose>0 0 1.0 0 0 0</pose>   <!-- 只给激光传感器加本地偏移：x y z R P Y -->
+        <pose>0 0 0 0 0 0</pose>   <!-- 只给激光传感器加本地偏移：x y z R P Y -->
         <topic>scan</topic>
         <update_rate>30</update_rate> <!-- 激光雷达更新频率 -->
@@ -31,5 +31,5 @@
             <range>
             <min>0.1</min>
-            <max>50.0</max>
+            <max>10.0</max>
             <resolution>0.01</resolution>
             </range>

File: ROS2/src/sim03_gazebo_classic/urdf/urdf/corn_harvester.urdf (robot description, URDF)
Before this commit: robot corn_harvester, 7 links, 6 joints
Links:
- link base_link: mass 10.2316767990512 -> 83.037
- link laser_link: mass 0.1 -> 0; geometry collision mesh filename=package://sim03_gazebo_classic/meshes/laser_link.STL; visual mesh filename=package://sim03_gazebo_classic/meshes/laser_link.STL
- link left_front_wheel_link0: mass 0.503853041294886 -> 0.98793
- link left_rear_wheel_link3: mass 0.503852022031433 -> 0.98793
- link right_front_wheel_link1: mass 0.503852021760132 -> 0.98793
- link right_rear_wheel_link2: mass 0.503853041294886 -> 0.98793
Joints:
- removed joint base_joint
- removed joint laser_joint
- added joint base_mount: type fixed, parent base_footprint, child base_link, origin xyz=0.0 0.0 0.06
- added joint laser_mount: type fixed, parent base_link, child laser_link, origin xyz=0 0.25 0.43 rpy=-1.5708 0 -1.5708, axis 0 0 0
- joint left_front_wheel_joint0: origin xyz=2.767 -3.5054 -1.1624 rpy=-1.5708 0 3.1416 -> xyz=-0.09 0.3 0.03 rpy=1.5708 0 0
- joint left_rear_wheel_joint3: origin xyz=2.767 2.3546 -1.1624 rpy=-1.5708 0 3.1416 -> xyz=-0.09 -0.3 0.03 rpy=1.5708 0 0
- joint right_front_wheel_joint1: axis 1 0 0 -> -1 0 0; origin xyz=-2.767 -3.5054 -1.4431 rpy=1.5708 0 0 -> xyz=0.09 0.3 0.03 rpy=1.5708 0 3.1416
- joint right_rear_wheel_joint2: axis 1 0 0 -> -1 0 0; origin xyz=-2.767 2.3546 -1.4431 rpy=1.5708 0 0 -> xyz=0.09 -0.3 0.03 rpy=1.5708 0 3.1416

Commit message: update

File: ROS2/src/sim01_urdf/urdf/urdf/corn_harvester.urdf (robot description, URDF)
Before this commit: robot corn_harvester, 7 links, 6 joints
Joints:
- joint base_mount: origin xyz=0.0 0.0 0.06 -> xyz=0.0 0.0 0.06 rpy=0 0 0
- joint left_front_wheel_joint0: axis -1 0 0 -> 1 0 0
- joint left_rear_wheel_joint3: axis -1 0 0 -> 1 0 0

File: ROS2/src/sim01_urdf/urdf/xacro/gazebo/move_control.urdf.xacro (robot description, xacro)
@@ -19,8 +19,8 @@
             <max_angular_acceleration>10</max_angular_acceleration>
             <min_angular_acceleration>-10</min_angular_acceleration>
-            <max_linear_velocity>0.5</max_linear_velocity>
-            <min_linear_velocity>-0.5</min_linear_velocity>
-            <max_angular_velocity>1</max_angular_velocity>
-            <min_angular_velocity>-1</min_angular_velocity>
+            <max_linear_velocity>2.0</max_linear_velocity>
+            <min_linear_velocity>-2.0</min_linear_velocity>
+            <max_angular_velocity>3.0</max_angular_velocity>
+            <min_angular_velocity>-3.0</min_angular_velocity>
         </plugin>
     </gazebo>

File: ROS2/src/sim01_urdf/urdf/xacro/gazebo/sensors_plugin.urdf.xacro (robot description, xacro)
@@ -30,6 +30,6 @@
             </scan>
             <range>
-            <min>0.1</min>
-            <max>10.0</max>
+            <min>0.15</min>
+            <max>6.0</max>
             <resolution>0.01</resolution>
             </range>
